Commit message: Normalize wheel joint axes in rover_test_description
The raw CAD export gave left-side wheel joints axis (-1,0,0) and right-side
wheel joints axis (1,0,0) -- opposite vectors, since SolidWorks assigns each
joint's axis independently per mate on a mirrored assembly. Practical effect:
driving straight required a [-,-,+,+] command pattern instead of a uniform
array, since same-signed commands on mirrored axes spin wheels in physically
opposite directions. Normalized all four to (1,0,0) so a single consistent
command sign drives all wheels the same physical direction.

Co-Authored-By: Claude Sonnet 5 <noreply@anthropic.com>

File: rover_ws/src/rover_test_description/urdf/rover_test.xacro (robot description, xacro)
@@ -197,5 +197,5 @@
   <parent link="front_left_steer_link"/>
   <child link="front_left_wheel_link"/>
-  <axis xyz="-1.0 -0.0 -0.0"/>
+  <axis xyz="1.0 0.0 0.0"/>
 </joint>
 <joint name="rear_left_wheel_joint" type="continuous">
@@ -203,5 +203,5 @@
   <parent link="rear_left_steer_link"/>
   <child link="rear_left_wheel_link"/>
-  <axis xyz="-1.0 0.0 0.0"/>
+  <axis xyz="1.0 0.0 0.0"/>
 </joint>
 <joint name="front_right_wheel_joint" type="continuous">
@@ -209,5 +209,5 @@
   <parent link="front_right_steer_link"/>
   <child link="front_right_wheel_link"/>
-  <axis xyz="1.0 -0.0 0.0"/>
+  <axis xyz="1.0 0.0 0.0"/>
 </joint>
 <joint name="rear_right_wheel_joint" type="continuous">
@@ -215,5 +215,5 @@
   <parent link="rear_right_steer_link"/>
   <child link="rear_right_wheel_link"/>
-  <axis xyz="1.0 -0.0 -0.0"/>
+  <axis xyz="1.0 0.0 0.0"/>
 </joint>
 <joint name="front_left_steer_joint" type="continuous">
