Commit message: Fold CAD-derived chassis geometry from rover_test_description into rover_description
rover_test_description's swerve driving was validated in Gazebo, so the
CAD geometry (meshes, real link/joint layout, gz_ros2_control wiring) no
longer needs to stay separate from rover_description, the package Nav2/
sim/mission work is meant to build against. Moves the meshes and CAD
xacro content over, adds a display.launch.py + rviz config so the model
can still be eyeballed without Gazebo, and removes rover_test_description
since nothing it provided is unique anymore.

Also fixes a pre-existing bug in rover_description/launch/gazebo.launch.py
(robot_description passed as a bare Command substitution instead of
ParameterValue(..., value_type=str), which fails to launch) -- this was
never exercised before since driving was only ever tested through
rover_test_description's launch file. Verified end-to-end post-fix: model
spawns, controllers activate, and /cmd_vel drives all four real wheels.

swerve_kinematics_node.py's hardcoded WHEEL_BASE/WHEEL_SEPARATION/
WHEEL_RADIUS still reflect the old placeholder chassis, not this CAD
geometry's actual (asymmetric) module layout -- left a TODO with the real
per-corner numbers rather than guessing at a fix, since the axis
convention doesn't map over directly. Needs a real look before trusting
/cmd_vel-driven turning on this geometry.

CLAUDE.md updated to match, including that this CAD export is itself
still an interim placeholder, not final chassis geometry.

Co-Authored-By: Claude Sonnet 5 <noreply@anthropic.com>

File: rover_ws/src/rover_description/urdf/materials.xacro (robot description, xacro)
@@ -1,4 +1,4 @@
 <?xml version="1.0" ?>
-<robot name="rover_test" xmlns:xacro="http://www.ros.org/wiki/xacro" >
+<robot name="rover" xmlns:xacro="http://www.ros.org/wiki/xacro" >
 <material name="silver">
   <color rgba="0.700 0.700 0.700 1.000"/>

File: rover_ws/src/rover_description/urdf/rover.urdf.xacro (robot description, xacro)
@@ -2,9 +2,18 @@
 <robot name="rover" xmlns:xacro="http://www.ros.org/wiki/xacro">
   <!--
-    Placeholder geometry only, to wire up and test the Gazebo + ros2_control +
-    Nav2 pipeline before a real chassis model exists. Replace the box/cylinder
-    links below with real geometry when ready; keep the steer/wheel joint
-    names in sync with config/rover_controllers.yaml and
-    rover_swerve_controller/swerve_kinematics_node.py if you rename them.
+    Chassis geometry (base_link + 4x swerve module meshes below) comes from
+    an early CAD export (SolidWorks-to-URDF), not the finalized rover
+    design — expect these meshes, masses, and joint origins to change again
+    as the real chassis design is finished. This replaced the box/cylinder
+    placeholder that used to live here (see git history), which was step
+    one of two: first wire up Gazebo + ros2_control + Nav2 against
+    *something*, then swap in CAD geometry once it existed. This is that
+    swap. It is NOT the final step — treat every dimension here as
+    provisional until it comes from released-for-manufacture CAD.
+    Link/joint names, the ros2_control block, and the Gazebo plugin/material
+    wiring were written by hand to match this project's Gazebo Harmonic +
+    gz_ros2_control stack; they must stay in sync with
+    config/rover_controllers.yaml and
+    rover_swerve_controller/swerve_kinematics_node.py if renamed.
     Swerve drivetrain: 4 independently-steerable wheel modules. Each module
     is a steer joint (vertical pivot) with a wheel joint (rolling axis) as
@@ -14,111 +23,252 @@
     node in the rover_swerve_controller package that converts /cmd_vel into
     per-module steer-angle + wheel-speed commands.
+    NOTE: rover_swerve_controller/swerve_kinematics_node.py still hardcodes
+    wheel radius and module positions from the old box/cylinder placeholder
+    (WHEEL_BASE=0.4, WHEEL_SEPARATION=0.5, WHEEL_RADIUS=0.15). Those no
+    longer match this CAD geometry's actual per-corner joint origins below
+    and need to be re-derived before trusting /cmd_vel-driven turning
+    behavior against this model — see the TODO in that file.
   -->
-  <xacro:property name="chassis_length" value="0.6"/>
-  <xacro:property name="chassis_width" value="0.4"/>
-  <xacro:property name="chassis_height" value="0.2"/>
-  <xacro:property name="wheel_radius" value="0.15"/>
-  <xacro:property name="wheel_width" value="0.08"/>
-  <xacro:property name="wheel_separation" value="0.5"/>
-  <xacro:property name="wheel_base" value="0.4"/>
-  <xacro:property name="steer_housing_radius" value="0.05"/>
-  <xacro:property name="steer_housing_height" value="0.08"/>
-  <material name="chassis_grey">
-    <color rgba="0.3 0.3 0.3 1"/>
-  </material>
-  <material name="wheel_black">
-    <color rgba="0.1 0.1 0.1 1"/>
-  </material>
-  <link name="base_link"/>
-  <joint name="chassis_joint" type="fixed">
-    <parent link="base_link"/>
-    <child link="chassis_link"/>
-    <origin xyz="0 0 ${wheel_radius}" rpy="0 0 0"/>
-  </joint>
-  <link name="chassis_link">
-    <visual>
-      <geometry>
-        <box size="${chassis_length} ${chassis_width} ${chassis_height}"/>
-      </geometry>
-      <material name="chassis_grey"/>
-    </visual>
-    <collision>
-      <geometry>
-        <box size="${chassis_length} ${chassis_width} ${chassis_height}"/>
-      </geometry>
-    </collision>
-    <inertial>
-      <mass value="15.0"/>
-      <inertia ixx="0.3" ixy="0.0" ixz="0.0" iyy="0.5" iyz="0.0" izz="0.6"/>
-    </inertial>
-  </link>
-  <!--
-    Swerve module: a steer joint (vertical pivot, rotates the whole module
-    about Z) with a wheel joint as its child (spins the wheel about its own
-    rolling axis). The wheel joint's origin is defined relative to the steer
-    link, so it stays correctly oriented no matter what angle the module is
-    currently steered to.
-  -->
-  <xacro:macro name="swerve_module" params="prefix x_reflect y_reflect">
-    <joint name="${prefix}_steer_joint" type="continuous">
-      <parent link="base_link"/>
-      <child link="${prefix}_steer_link"/>
-      <origin xyz="${x_reflect * wheel_base / 2} ${y_reflect * wheel_separation / 2} ${wheel_radius}" rpy="0 0 0"/>
-      <axis xyz="0 0 1"/>
-    </joint>
-    <link name="${prefix}_steer_link">
-      <visual>
-        <geometry>
-          <cylinder radius="${steer_housing_radius}" length="${steer_housing_height}"/>
-        </geometry>
-        <material name="chassis_grey"/>
-      </visual>
-      <collision>
-        <geometry>
-          <cylinder radius="${steer_housing_radius}" length="${steer_housing_height}"/>
-        </geometry>
-      </collision>
-      <inertial>
-        <mass value="0.5"/>
-        <inertia ixx="0.001" ixy="0.0" ixz="0.0" iyy="0.001" iyz="0.0" izz="0.001"/>
-      </inertial>
-    </link>
-    <joint name="${prefix}_wheel_joint" type="continuous">
-      <parent link="${prefix}_steer_link"/>
-      <child link="${prefix}_wheel_link"/>
-      <origin xyz="0 0 0" rpy="${-pi/2} 0 0"/>
-      <axis xyz="0 0 1"/>
-    </joint>
-    <link name="${prefix}_wheel_link">
-      <visual>
-        <geometry>
-          <cylinder radius="${wheel_radius}" length="${wheel_width}"/>
-        </geometry>
-        <material name="wheel_black"/>
-      </visual>
-      <collision>
-        <geometry>
-          <cylinder radius="${wheel_radius}" length="${wheel_width}"/>
-        </geometry>
-      </collision>
-      <inertial>
-        <mass value="1.5"/>
-        <inertia ixx="0.01" ixy="0.0" ixz="0.0" iyy="0.01" iyz="0.0" izz="0.015"/>
-      </inertial>
-    </link>
-  </xacro:macro>
-  <xacro:swerve_module prefix="front_left" x_reflect="1" y_reflect="1"/>
-  <xacro:swerve_module prefix="front_right" x_reflect="1" y_reflect="-1"/>
-  <xacro:swerve_module prefix="rear_left" x_reflect="-1" y_reflect="1"/>
-  <xacro:swerve_module prefix="rear_right" x_reflect="-1" y_reflect="-1"/>
+  <xacro:include filename="$(find rover_description)/urdf/materials.xacro" />
+  <xacro:include filename="$(find rover_description)/urdf/rover.gazebo" />
+  <link name="base_link">
+    <inertial>
+      <origin xyz="1.7662172446492366e-08 0.04237215152825712 0.09216107589120397" rpy="0 0 0"/>
+      <mass value="595.1849542563896"/>
+      <inertia ixx="19.500193" iyy="39.83973" izz="55.970633" ixy="1e-06" iyz="-0.807843" ixz="0.0"/>
+    </inertial>
+    <visual>
+      <origin xyz="0 0 0" rpy="0 0 0"/>
+      <geometry>
+        <mesh filename="file://$(find rover_description)/meshes/base_link.stl" scale="0.001 0.001 0.001"/>
+      </geometry>
+      <material name="silver"/>
+    </visual>
+    <collision>
+      <origin xyz="0 0 0" rpy="0 0 0"/>
+      <geometry>
+        <mesh filename="file://$(find rover_description)/meshes/base_link.stl" scale="0.001 0.001 0.001"/>
+      </geometry>
+    </collision>
+  </link>
+  <link name="front_left_wheel_link">
+    <inertial>
+      <origin xyz="0.0507999999999999 -1.1102230246251565e-16 5.551115123125783e-17" rpy="0 0 0"/>
+      <mass value="25.864295489856012"/>
+      <inertia ixx="0.133493" iyy="0.088995" izz="0.088995" ixy="-0.0" iyz="0.0" ixz="0.0"/>
+    </inertial>
+    <visual>
+      <origin xyz="-0.3556 0.3175 0.1905" rpy="0 0 0"/>
+      <geometry>
+        <mesh filename="file://$(find rover_description)/meshes/wheel1_1.stl" scale="0.001 0.001 0.001"/>
+      </geometry>
+      <material name="silver"/>
+    </visual>
+    <collision>
+      <origin xyz="-0.3556 0.3175 0.1905" rpy="0 0 0"/>
+      <geometry>
+        <mesh filename="file://$(find rover_description)/meshes/wheel1_1.stl" scale="0.001 0.001 0.001"/>
+      </geometry>
+    </collision>
+  </link>
+  <link name="rear_left_wheel_link">
+    <inertial>
+      <origin xyz="0.050799999999999956 1.1102230246251565e-16 3.885780586188048e-16" rpy="0 0 0"/>
+      <mass value="25.864295489856012"/>
+      <inertia ixx="0.133493" iyy="0.088995" izz="0.088995" ixy="0.0" iyz="0.0" ixz="0.0"/>
+    </inertial>
+    <visual>
+      <origin xyz="-0.3556 -0.2921 0.1905" rpy="0 0 0"/>
+      <geometry>
+        <mesh filename="file://$(find rover_description)/meshes/wheel3_1.stl" scale="0.001 0.001 0.001"/>
+      </geometry>
+      <material name="silver"/>
+    </visual>
+    <collision>
+      <origin xyz="-0.3556 -0.2921 0.1905" rpy="0 0 0"/>
+      <geometry>
+        <mesh filename="file://$(find rover_description)/meshes/wheel3_1.stl" scale="0.001 0.001 0.001"/>
+      </geometry>
+    </collision>
+  </link>
+  <link name="front_right_wheel_link">
+    <inertial>
+      <origin xyz="-0.050799999999999845 -3.6637359812630166e-15 -2.7755575615628914e-16" rpy="0 0 0"/>
+      <mass value="25.864295489856012"/>
+      <inertia ixx="0.133493" iyy="0.088995" izz="0.088995" ixy="-0.0" iyz="-0.0" ixz="0.0"/>
+    </inertial>
+    <visual>
+      <origin xyz="0.3556 0.3175 0.1905" rpy="0 0 0"/>
+      <geometry>
+        <mesh filename="file://$(find rover_description)/meshes/wheel2_1.stl" scale="0.001 0.001 0.001"/>
+      </geometry>
+      <material name="silver"/>
+    </visual>
+    <collision>
+      <origin xyz="0.3556 0.3175 0.1905" rpy="0 0 0"/>
+      <geometry>
+        <mesh filename="file://$(find rover_description)/meshes/wheel2_1.stl" scale="0.001 0.001 0.001"/>
+      </geometry>
+    </collision>
+  </link>
+  <link name="rear_right_wheel_link">
+    <inertial>
+      <origin xyz="-0.05080000000000029 -3.7192471324942744e-15 1.6653345369377348e-16" rpy="0 0 0"/>
+      <mass value="25.864295489856012"/>
+      <inertia ixx="0.133493" iyy="0.088995" izz="0.088995" ixy="0.0" iyz="0.0" ixz="0.0"/>
+    </inertial>
+    <visual>
+      <origin xyz="0.3556 -0.2921 0.1905" rpy="0 0 0"/>
+      <geometry>
+        <mesh filename="file://$(find rover_description)/meshes/wheel4_1.stl" scale="0.001 0.001 0.001"/>
+      </geometry>
+      <material name="silver"/>
+    </visual>
+    <collision>
+      <origin xyz="0.3556 -0.2921 0.1905" rpy="0 0 0"/>
+      <geometry>
+        <mesh filename="file://$(find rover_description)/meshes/wheel4_1.stl" scale="0.001 0.001 0.001"/>
+      </geometry>
+    </collision>
+  </link>
+  <link name="front_left_steer_link">
+    <inertial>
+      <origin xyz="-0.004588209054589121 -1.1102230246251565e-16 -0.0951512261261479" rpy="0 0 0"/>
+      <mass value="11.71442300300121"/>
+      <inertia ixx="0.072711" iyy="0.074344" izz="0.018661" ixy="0.0" iyz="-0.0" ixz="-0.013033"/>
+    </inertial>
+    <visual>
+      <origin xyz="-0.3556 0.3175 -0.0254" rpy="0 0 0"/>
+      <geometry>
+        <mesh filename="file://$(find rover_description)/meshes/mount1_1.stl" scale="0.001 0.001 0.001"/>
+      </geometry>
+      <material name="silver"/>
+    </visual>
+    <collision>
+      <origin xyz="-0.3556 0.3175 -0.0254" rpy="0 0 0"/>
+      <geometry>
+        <mesh filename="file://$(find rover_description)/meshes/mount1_1.stl" scale="0.001 0.001 0.001"/>
+      </geometry>
+    </collision>
+  </link>
+  <link name="front_right_steer_link">
+    <inertial>
+      <origin xyz="0.00458820905458901 5.551115123125783e-17 -0.09515122612614813" rpy="0 0 0"/>
+      <mass value="11.714423003001206"/>
+      <inertia ixx="0.072711" iyy="0.074344" izz="0.018661" ixy="0.0" iyz="0.0" ixz="0.013033"/>
+    </inertial>
+    <visual>
+      <origin xyz="0.3556 0.3175 -0.0254" rpy="0 0 0"/>
+      <geometry>
+        <mesh filename="file://$(find rover_description)/meshes/mount2_1.stl" scale="0.001 0.001 0.001"/>
+      </geometry>
+      <material name="silver"/>
+    </visual>
+    <collision>
+      <origin xyz="0.3556 0.3175 -0.0254" rpy="0 0 0"/>
+      <geometry>
+        <mesh filename="file://$(find rover_description)/meshes/mount2_1.stl" scale="0.001 0.001 0.001"/>
+      </geometry>
+    </collision>
+  </link>
+  <link name="rear_left_steer_link">
+    <inertial>
+      <origin xyz="-0.00458820905458901 1.1102230246251565e-16 -0.09515122612614782" rpy="0 0 0"/>
+      <mass value="11.71442300300121"/>
+      <inertia ixx="0.072711" iyy="0.074344" izz="0.018661" ixy="0.0" iyz="0.0" ixz="-0.013033"/>
+    </inertial>
+    <visual>
+      <origin xyz="-0.3556 -0.2921 -0.0254" rpy="0 0 0"/>
+      <geometry>
+        <mesh filename="file://$(find rover_description)/meshes/mount3_1.stl" scale="0.001 0.001 0.001"/>
+      </geometry>
+      <material name="silver"/>
+    </visual>
+    <collision>
+      <origin xyz="-0.3556 -0.2921 -0.0254" rpy="0 0 0"/>
+      <geometry>
+        <mesh filename="file://$(find rover_description)/meshes/mount3_1.stl" scale="0.001 0.001 0.001"/>
+      </geometry>
+    </collision>
+  </link>
+  <link name="rear_right_steer_link">
+    <inertial>
+      <origin xyz="0.004588209054588566 -5.551115123125783e-17 -0.09515122612614793" rpy="0 0 0"/>
+      <mass value="11.71442300300121"/>
+      <inertia ixx="0.072711" iyy="0.074344" izz="0.018661" ixy="0.0" iyz="0.0" ixz="0.013033"/>
+    </inertial>
+    <visual>
+      <origin xyz="0.3556 -0.2921 -0.0254" rpy="0 0 0"/>
+      <geometry>
+        <mesh filename="file://$(find rover_description)/meshes/mount4_1.stl" scale="0.001 0.001 0.001"/>
+      </geometry>
+      <material name="silver"/>
+    </visual>
+    <collision>
+      <origin xyz="0.3556 -0.2921 -0.0254" rpy="0 0 0"/>
+      <geometry>
+        <mesh filename="file://$(find rover_description)/meshes/mount4_1.stl" scale="0.001 0.001 0.001"/>
+      </geometry>
+    </collision>
+  </link>
+  <joint name="front_left_wheel_joint" type="continuous">
+    <origin xyz="0.0 0.0 -0.2159" rpy="0 0 0"/>
+    <parent link="front_left_steer_link"/>
+    <child link="front_left_wheel_link"/>
+    <axis xyz="1.0 0.0 0.0"/>
+  </joint>
+  <joint name="rear_left_wheel_joint" type="continuous">
+    <origin xyz="0.0 0.0 -0.2159" rpy="0 0 0"/>
+    <parent link="rear_left_steer_link"/>
+    <child link="rear_left_wheel_link"/>
+    <axis xyz="1.0 0.0 0.0"/>
+  </joint>
+  <joint name="front_right_wheel_joint" type="continuous">
+    <origin xyz="0.0 0.0 -0.2159" rpy="0 0 0"/>
+    <parent link="front_right_steer_link"/>
+    <child link="front_right_wheel_link"/>
+    <axis xyz="1.0 0.0 0.0"/>
+  </joint>
+  <joint name="rear_right_wheel_joint" type="continuous">
+    <origin xyz="0.0 0.0 -0.2159" rpy="0 0 0"/>
+    <parent link="rear_right_steer_link"/>
+    <child link="rear_right_wheel_link"/>
+    <axis xyz="1.0 0.0 0.0"/>
+  </joint>
+  <joint name="front_left_steer_joint" type="continuous">
+    <origin xyz="0.3556 -0.3175 0.0254" rpy="0 0 0"/>
+    <parent link="base_link"/>
+    <child link="front_left_steer_link"/>
+    <axis xyz="0.0 0.0 1.0"/>
+  </joint>
+  <joint name="front_right_steer_joint" type="continuous">
+    <origin xyz="-0.3556 -0.3175 0.0254" rpy="0 0 0"/>
+    <parent link="base_link"/>
+    <child link="front_right_steer_link"/>
+    <axis xyz="0.0 0.0 1.0"/>
+  </joint>
+  <joint name="rear_left_steer_joint" type="continuous">
+    <origin xyz="0.3556 0.2921 0.0254" rpy="0 0 0"/>
+    <parent link="base_link"/>
+    <child link="rear_left_steer_link"/>
+    <axis xyz="0.0 0.0 1.0"/>
+  </joint>
+  <joint name="rear_right_steer_joint" type="continuous">
+    <origin xyz="-0.3556 0.2921 0.0254" rpy="0 0 0"/>
+    <parent link="base_link"/>
+    <child link="rear_right_steer_link"/>
+    <axis xyz="0.0 0.0 1.0"/>
+  </joint>
+  <!-- Sensor mount points are placeholders (not yet taken from real CAD
+       mount locations) — revisit once the chassis design settles. -->
   <joint name="lidar_joint" type="fixed">
-    <parent link="chassis_link"/>
+    <parent link="base_link"/>
     <child link="lidar_link"/>
-    <origin xyz="0 0 ${chassis_height / 2 + 0.05}" rpy="0 0 0"/>
+    <origin xyz="0 0 0.25" rpy="0 0 0"/>
   </joint>
   <link name="lidar_link">
     <visual>
       <geometry><cylinder radius="0.04" length="0.06"/></geometry>
-      <material name="wheel_black"/>
+      <material name="silver"/>
     </visual>
     <collision>
@@ -133,12 +283,12 @@
        slam_toolbox is the near-term priority per CLAUDE.md's SLAM go/no-go plan. -->
   <joint name="camera_joint" type="fixed">
-    <parent link="chassis_link"/>
+    <parent link="base_link"/>
     <child link="camera_link"/>
-    <origin xyz="${chassis_length / 2} 0 0.05" rpy="0 0 0"/>
+    <origin xyz="0.35 0 0.1" rpy="0 0 0"/>
   </joint>
   <link name="camera_link">
     <visual>
       <geometry><box size="0.03 0.09 0.03"/></geometry>
-      <material name="chassis_grey"/>
+      <material name="silver"/>
     </visual>
     <collision>
